File: Cadsoft Eagle and PCB Fab Class/Eagle Files/familab_pov_finished/familab_pov_finished.sch (EAGLE design)
At the start: 10 parts, among them U1 Tiny85-20-SMT

Commit message: Increased Dimensions slightly and Fixed Arduino Code
Parts:
- J1: device fri-001:JUMPERSIDE -> pov_class:JUMPERSIDE
Changed lines of the file:
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@@
 <?xml version="1.0" encoding="utf-8"?>
 <!DOCTYPE eagle SYSTEM "eagle.dtd">
-<eagle version="6.5.0">
+<eagle version="6.4">
 <drawing>
 <settings>
@@
 <part name="P+2" library="supply1" deviceset="VCC" device=""/>
 <part name="GND3" library="supply1" deviceset="GND" device=""/>
-<part name="J1" library="fri-001" deviceset="JUMPER" device="SIDE"/>
+<part name="J1" library="pov_class" deviceset="JUMPER" device="SIDE"/>
 <part name="U$2" library="pov_class" deviceset="MOUNTING_PAD" device=""/>
 <part name="P+3" library="supply1" deviceset="VCC" device=""/>

Commit message: Updates
Parts:
- J1: device pov_class:JUMPERSIDE -> pov_class_finished:JUMPERSIDE
- U$4: device pov_class:ICSP_PROGRAM -> pov_class_finished:ICSP_PROGRAM
Changed lines of the file:
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@@
 <?xml version="1.0" encoding="utf-8"?>
 <!DOCTYPE eagle SYSTEM "eagle.dtd">
-<eagle version="6.4">
+<eagle version="6.5.0">
 <drawing>
 <settings>
@@
 <part name="P+2" library="supply1" deviceset="VCC" device=""/>
 <part name="GND3" library="supply1" deviceset="GND" device=""/>
-<part name="J1" library="pov_class" deviceset="JUMPER" device="SIDE"/>
+<part name="J1" library="pov_class_finished" deviceset="JUMPER" device="SIDE"/>
 <part name="U$2" library="pov_class" deviceset="MOUNTING_PAD" device=""/>
 <part name="P+3" library="supply1" deviceset="VCC" device=""/>
 <part name="GND4" library="supply1" deviceset="GND" device=""/>
-<part name="U$4" library="pov_class" deviceset="ICSP_PROGRAM" device=""/>
+<part name="U$4" library="pov_class_finished" deviceset="ICSP_PROGRAM" device=""/>
 </parts>
 <sheets>
